File: Relay_board_kiCad_v2/Relay_board_v2.kicad_pcb (KiCad board)
At the start: 2 copper layers, 74.5 x 63 mm, 33 parts, among them J1 Conn_01x03_Pin, J2 Conn_01x03_Pin, J3 Conn_01x03_Pin, J4 Conn_01x03_Pin, J5 Conn_01x06_Pin, K1 SANYOU_SRD_Form_C, K2 SANYOU_SRD_Form_C, K3 SANYOU_SRD_Form_C, K4 SANYOU_SRD_Form_C, Q1 BC817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

Commit message: Add files via upload
pinout replacement
Parts:
- J5: footprint Connector_PinHeader_2.00mm:PinHeader_1x06_P2.00mm_Vertical -> Connector_PinHeader_2.54mm:PinHeader_1x06_P2.54mm_Vertical
- moved J5 1.55 mm to (116.2, 101.8)
Routing:
- net VCC: track 183.6 -> 182.5 mm
- net /IN1: track 26.1 -> 25.3 mm
- net GND: track 90.3 -> 91.0 mm
